File: PCB/therick64BA.kicad_pcb (KiCad board)
At the start: 2 copper layers, 312.7 x 76.7 mm, 160 parts, among them J1 TYPE-C-31-M12_13, J2 AVR-ISP-6, K1 KEYSW, K10 KEYSW, K11 KEYSW, K12 KEYSW, K13 KEYSW, K14 KEYSW, K15 KEYSW, K16 KEYSW, K17 KEYSW, K18 KEYSW, K19 KEYSW, K2 KEYSW, K20 KEYSW, K21 KEYSW, K22 KEYSW, K23 KEYSW, K24 KEYSW, K25 KEYSW, K26 KEYSW, K27 KEYSW, K28 KEYSW, K29 KEYSW, K3 KEYSW, K30 KEYSW, K31 KEYSW, K32 KEYSW, K33 KEYSW, K34 KEYSW, K35 KEYSW, K36 KEYSW, K37 KEYSW, K38 KEYSW, K39 KEYSW, K4 KEYSW, K40 KEYSW, K41 KEYSW, K42 KEYSW, K43 KEYSW, K44 KEYSW, K45 KEYSW, K46 KEYSW, K47 KEYSW, K48 KEYSW, K49 KEYSW, K5 KEYSW, K50 KEYSW, K51 KEYSW, K52 KEYSW, K53 KEYSW, K54 KEYSW, K55 KEYSW, K56 KEYSW, K57 KEYSW, K58 KEYSW, K59 KEYSW, K6 KEYSW, K60 KEYSW, K61 KEYSW, K62 KEYSW, K63 KEYSW, K64 KEYSW, K7 KEYSW, K8 KEYSW, K9 KEYSW, SW1 SW_PUSH, U1 ATMEGA32U4, U2 HOLE, U3 USBLC6-2SC6, Y1 16Mhz

Commit message: Update to 19mm
Parts:
- added U4: HOLE, Keeb_footprints:MouseBite_IPC7351, F.Cu at (272.8, 49.8)
- added U5: HOLE, Keeb_footprints:MouseBite_IPC7351, F.Cu at (272.8, 96.1)
- added U6: HOLE, Keeb_footprints:MouseBite_IPC7351, F.Cu at (272.8, 65.0)
- added U7: HOLE, Keeb_footprints:MouseBite_IPC7351, F.Cu at (272.8, 81.3)
- added U8: HOLE, Artwork:QMKBadgeSmall, B.Cu at (197.1, 94.0)
- J1: footprint random-keyboard-parts:TYPE-C-31-M-12 -> Keeb_footprints:TYPE-C-31-M-12
- K1, K10, K11, K12, K13, K14, K15, K16, K17, K18, K19, K2, K20, K21, K22, K23, K24, K25, K26, K27, K28, K29, K3, K30, K31, K32, K33, K34, K35, K36, K37, K38, K39, K4, K40, K41, K42, K43, K44, K45, K46, K47, K48, K49, K5, K50, K51, K52, K53, K54, K55, K56, K57, K58, K59, K6, K60, K61, K62, K63, K64, K7, K8, K9: footprint acheron_MX:MX100 -> Keeb_footprints:MX100
- U3: footprint Package_TO_SOT_SMD:SOT-23-6 -> acheron_Components:SOT-23-6
- Y1: value 16Mhz -> 16MHz
- moved U2 18.1 mm to (237.6, 76.0)
- moved J2 0.97 mm to (121.8, 55.2)
- moved R1 0.89 mm to (73.4, 72.4)
- moved J1 0.78 mm to (84.0, 41.2)
- moved RCC1 0.73 mm to (77.5, 40.9)
- moved RCC2 0.73 mm to (90.5, 40.9)
- moved D11 0.63 mm to (253.4, 43.3)
- moved D12 0.63 mm to (256.5, 43.3)
- moved D23 0.63 mm to (253.4, 62.3)
- moved D24 0.63 mm to (256.5, 62.3)
- moved D35 0.63 mm to (253.4, 81.4)
- moved D36 0.63 mm to (256.5, 81.4)
- moved D47 0.63 mm to (253.4, 100.4)
- moved D48 0.63 mm to (256.5, 100.4)
- moved K48 0.63 mm to (264.5, 101.4), turned to 0 degrees
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Connections:
- net UCap renamed GND
Routing:
- net row1: track 327.0 -> 305.2 mm
- net Net-(D37-Pad2): track 14.6 -> 21.9 mm
- net col2: track 74.2 -> 79.4 mm
- net row0: track 345.4 -> 349.3 mm
- net row2: track 432.4 -> 428.7 mm
- net col15: track 392.9 -> 395.6 mm
- net VCC: track 144.6 -> 146.7 mm
- net D+BUS: track 8.76 -> 6.75 mm
- net col12: track 331.7 -> 329.7 mm
- net col14: track 370.5 -> 368.8 mm
- net col11: track 258.3 -> 256.7 mm
- net col3: track 106.3 -> 104.6 mm
- net GND: track 14.9 -> 13.3 mm
- net ISP_Reset: track 63.6 -> 64.9 mm
- net row3: track 330.8 -> 332.0 mm
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Other:
- board size 312.7 x 76.7 mm -> 312.4 x 75.8 mm
- board text added: "16MHz"
- board text added: "therick"
- board text added: "therick64BA_19mm"
- board text removed: "16Mhz"
- board text removed: "therick64"

Commit message: Update some routing
Routing:
- net VCC: track 146.7 -> 144.8 mm
Changed lines of the file:
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@@
     (thickness 1.6)
     (drawings 78)
-    (tracks 823)
+    (tracks 821)
     (zones 0)
     (modules 165)
@@
   )
   (module Keeb_footprints:MouseBite_IPC7351 (layer F.Cu)
-    (at 272.84 49.78 90)
-    (fp_text reference U4 (at 0 -2.8 90) (layer Dwgs.User)
+    (at 272.84 96.14 90)
+    (fp_text reference U5 (at -0.508 -2.8 90) (layer Cmts.User)
       (effects (font (size 1 1) (thickness 0.15)))
     )
-    (fp_text value HOLE (at 0 -1.27 90) (layer F.Fab)
+    (fp_text value HOLE (at -0.381 -1.143 90) (layer F.Fab)
       (effects (font (size 1 1) (thickness 0.15)))
     )
-    (pad "" np_thru_hole circle (at -3.048 0 90) (size 0.8 0.8) (drill 0.8) (layers *.Cu *.Mask))
+    (pad "" np_thru_hole circle (at -2.794 0 90) (size 0.8 0.8) (drill 0.8) (layers *.Cu *.Mask))
     (pad "" np_thru_hole circle (at -1.377 0 90) (size 0.8 0.8) (drill 0.8) (layers *.Cu *.Mask))
     (pad "" np_thru_hole circle (at 2.794 0 90) (size 0.8 0.8) (drill 0.8) (layers *.Cu *.Mask))
     (pad "" np_thru_hole circle (at 1.377 0 90) (size 0.8 0.8) (drill 0.8) (layers *.Cu *.Mask))
     (pad "" np_thru_hole circle (at 0 0 90) (size 0.8 0.8) (drill 0.8) (layers *.Cu *.Mask))
+    (pad "" np_thru_hole circle (at -4.191 0 90) (size 0.8 0.8) (drill 0.8) (layers *.Cu *.Mask))
+    (pad "" np_thru_hole circle (at 4.191 0 90) (size 0.8 0.8) (drill 0.8) (layers *.Cu *.Mask))
   )
   (module Keeb_footprints:MouseBite_IPC7351 (layer F.Cu)
-    (at 272.84 96.14 90)
-    (fp_text reference U5 (at -0.508 -2.8 90) (layer Cmts.User)
+    (at 272.84 49.78 90)
+    (fp_text reference U4 (at 0 -2.8 90) (layer Dwgs.User)
       (effects (font (size 1 1) (thickness 0.15)))
     )
-    (fp_text value HOLE (at -0.381 -1.143 90) (layer F.Fab)
+    (fp_text value HOLE (at 0 -1.27 90) (layer F.Fab)
       (effects (font (size 1 1) (thickness 0.15)))
     )
-    (pad "" np_thru_hole circle (at -2.794 0 90) (size 0.8 0.8) (drill 0.8) (layers *.Cu *.Mask))
+    (pad "" np_thru_hole circle (at -3.048 0 90) (size 0.8 0.8) (drill 0.8) (layers *.Cu *.Mask))
     (pad "" np_thru_hole circle (at -1.377 0 90) (size 0.8 0.8) (drill 0.8) (layers *.Cu *.Mask))
     (pad "" np_thru_hole circle (at 2.794 0 90) (size 0.8 0.8) (drill 0.8) (layers *.Cu *.Mask))
@@
   (segment (start 257.289 106.54) (end 261.94 106.54) (width 0.25) (layer B.Cu) (net 48))
   (segment (start 256.54 105.791) (end 257.289 106.54) (width 0.25) (layer B.Cu) (net 48))
-  (segment (start 88.1375 70.557402) (end 88.1375 69.875) (width 0.5) (layer B.Cu) (net 49))
-  (segment (start 88.1375 69.875) (end 88.1375 68.625) (width 0.5) (layer B.Cu) (net 49))
   (segment (start 81.153 59.563) (end 81.153 62.945) (width 0.25) (layer B.Cu) (net 49))
   (segment (start 107.47375 47.39375) (end 100.68825 47.39375) (width 0.25) (layer B.Cu) (net 49))
