File: PCB/therick64BA.kicad_pcb (KiCad board)
At the start: 2 copper layers, 312.4 x 75.8 mm, 165 parts, among them J1 TYPE-C-31-M12_13, J2 AVR-ISP-6, K1 KEYSW, K10 KEYSW, K11 KEYSW, K12 KEYSW, K13 KEYSW, K14 KEYSW, K15 KEYSW, K16 KEYSW, K17 KEYSW, K18 KEYSW, K19 KEYSW, K2 KEYSW, K20 KEYSW, K21 KEYSW, K22 KEYSW, K23 KEYSW, K24 KEYSW, K25 KEYSW, K26 KEYSW, K27 KEYSW, K28 KEYSW, K29 KEYSW, K3 KEYSW, K30 KEYSW, K31 KEYSW, K32 KEYSW, K33 KEYSW, K34 KEYSW, K35 KEYSW, K36 KEYSW, K37 KEYSW, K38 KEYSW, K39 KEYSW, K4 KEYSW, K40 KEYSW, K41 KEYSW, K42 KEYSW, K43 KEYSW, K44 KEYSW, K45 KEYSW, K46 KEYSW, K47 KEYSW, K48 KEYSW, K49 KEYSW, K5 KEYSW, K50 KEYSW, K51 KEYSW, K52 KEYSW, K53 KEYSW, K54 KEYSW, K55 KEYSW, K56 KEYSW, K57 KEYSW, K58 KEYSW, K59 KEYSW, K6 KEYSW, K60 KEYSW, K61 KEYSW, K62 KEYSW, K63 KEYSW, K64 KEYSW, K7 KEYSW, K8 KEYSW, K9 KEYSW, SW1 SW_PUSH, U1 ATMEGA32U4, U2 HOLE, U3 USBLC6-2SC6, U4 HOLE, U5 HOLE, U6 HOLE, U7 HOLE, U8 HOLE, Y1 16MHz

Commit message: Changed pins to make routing cleaner
Parts:
- removed U8: HOLE, Artwork:QMKBadgeSmall
- moved U5 0.76 mm to (273.6, 96.1)
- moved U6 0.76 mm to (273.6, 65.0)
- moved U4 0.76 mm to (273.6, 49.8)
- moved U7 0.76 mm to (273.6, 81.3)
- moved D13 0.51 mm to (63.5, 61.8)
- moved D14 0.51 mm to (66.7, 61.8)
- moved D15 0.51 mm to (101.6, 61.8)
- moved D16 0.51 mm to (104.8, 61.8)
- moved D17 0.51 mm to (139.7, 61.8)
- moved D18 0.51 mm to (142.9, 61.8)
- moved D19 0.51 mm to (177.4, 61.8)
- moved D20 0.51 mm to (180.6, 61.8)
- moved D21 0.51 mm to (215.4, 61.8)
- moved D22 0.51 mm to (218.6, 61.8)
- moved D23 0.51 mm to (253.4, 61.8)
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Connections:
- U1 pad 10: col4 -> col10
- U1 pad 11: col3 -> col11
- U1 pad 38: col11 -> col3
- U1 pad 39: col10 -> col4
- U1 pad 40: col9 -> col5
- U1 pad 41: col8 -> col6
- U1 pad 8: col6 -> col8
- U1 pad 9: col5 -> col9
Routing:
- net row2: track 428.7 -> 328.5 mm
- net col8: track 198.7 -> 183.5 mm, vias 2 -> 0
- net col10: track 238.3 -> 223.2 mm, vias 2 -> 0
- net col11: track 256.7 -> 242.2 mm, vias 2 -> 0
- net col9: track 218.1 -> 205.1 mm, vias 2 -> 0
- net VCC: track 144.8 -> 153.5 mm, vias 2 -> 6
- net Net-(D37-Pad2): track 21.9 -> 14.9 mm
- net XTAL2: track 18.4 -> 11.7 mm
- net col7: track 171.7 -> 166.0 mm
- net row3: track 332.0 -> 326.3 mm
- net col0: track 87.0 -> 82.5 mm
- net col2: track 79.4 -> 74.9 mm
- net col14: track 368.8 -> 365.3 mm
- net col15: track 395.6 -> 393.0 mm
- net col3: track 104.6 -> 106.9 mm, vias 0 -> 2
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Other:
- outline, holes or cut-outs redrawn
- board text added: "PCB Rev 1.0"
- board text added: "therick64BA"
- board text removed: "therick"
- board text removed: "therick64BA_19mm"
