File: PCB/therick64BA.sch (KiCad schematic (older format))
At the start: 160 parts, among them J1 TYPE-C-31-M12_13, J2 AVR-ISP-6, K1 KEYSW, K10 KEYSW, K11 KEYSW, K12 KEYSW, K13 KEYSW, K14 KEYSW, K15 KEYSW, K16 KEYSW, K17 KEYSW, K18 KEYSW, K19 KEYSW, K2 KEYSW, K20 KEYSW, K21 KEYSW, K22 KEYSW, K23 KEYSW, K24 KEYSW, K25 KEYSW, K26 KEYSW, K27 KEYSW, K28 KEYSW, K29 KEYSW, K3 KEYSW, K30 KEYSW, K31 KEYSW, K32 KEYSW, K33 KEYSW, K34 KEYSW, K35 KEYSW, K36 KEYSW, K37 KEYSW, K38 KEYSW, K39 KEYSW, K4 KEYSW, K40 KEYSW, K41 KEYSW, K42 KEYSW, K43 KEYSW, K44 KEYSW, K45 KEYSW, K46 KEYSW, K47 KEYSW, K48 KEYSW, K49 KEYSW, K5 KEYSW, K50 KEYSW, K51 KEYSW, K52 KEYSW, K53 KEYSW, K54 KEYSW, K55 KEYSW, K56 KEYSW, K57 KEYSW, K58 KEYSW, K59 KEYSW, K6 KEYSW, K60 KEYSW, K61 KEYSW, K62 KEYSW, K63 KEYSW, K64 KEYSW, K7 KEYSW, K8 KEYSW, K9 KEYSW, SW1 SW_PUSH, U1 ATMEGA32U4, U2 HOLE, U3 USBLC6-2SC6, Y1 16Mhz

Commit message: Update to 19mm
Parts:
- added U4, U5, U6, U7: HOLE, Keeb_footprints:MouseBite_IPC7351, symbol lets_split-cache:HOLE
- added U8: HOLE, Artwork:QMKBadgeSmall, symbol lets_split-cache:HOLE
- C1, C2, C3, C4, C5, CX1, CX2: symbol therick64BA-rescue:Device_C_Small-shark-cache-therick_v3-rescue-therick_v2-rescue-therick-rescue-therick64-rescue -> Device:C_Small
- J1: footprint random-keyboard-parts:TYPE-C-31-M-12 -> Keeb_footprints:TYPE-C-31-M-12
- K1, K10, K11, K12, K13, K14, K15, K16, K17, K18, K19, K2, K20, K21, K22, K23, K24, K25, K26, K27, K28, K29, K3, K30, K31, K32, K33, K34, K35, K36, K37, K38, K39, K4, K40, K41, K42, K43, K44, K45, K46, K47, K48, K49, K5, K50, K51, K52, K53, K54, K55, K56, K57, K58, K59, K6, K60, K61, K62, K63, K64, K7, K8, K9: footprint acheron_MX:MX100 -> Keeb_footprints:MX100
- U3: footprint Package_TO_SOT_SMD:SOT-23-6 -> acheron_Components:SOT-23-6
- Y1: value 16Mhz -> 16MHz
Other:
- note added: "Mouse bites"
- note added: "QMK"
- moved on the sheet: C1, C2, C3, C4, C5, CX1, CX2, U3, Y1

Commit message: Changed pins to make routing cleaner
Parts:
- removed U8: HOLE, Artwork:QMKBadgeSmall, symbol lets_split-cache:HOLE
Connections:
- net col10: now also U1.10 (PB2/MOSI); no longer U1.39 (PF4)
- net col11: now also U1.11 (PB3/MISO); no longer U1.38 (PF5)
- net col3: now also U1.38 (PF5); no longer U1.11 (PB3/MISO)
- net col4: now also U1.39 (PF4); no longer U1.10 (PB2/MOSI)
- net col5: now also U1.40 (PF1); no longer U1.9 (PB1/SCK)
- net col6: now also U1.41 (PF0); no longer U1.8 (PB0/SS)
- net col8: now also U1.8 (PB0/SS); no longer U1.41 (PF0)
- net col9: now also U1.9 (PB1/SCK); no longer U1.40 (PF1)
Other:
- note removed: "QMK"
- moved on the sheet: D1, D10, D11, D12, D13, D14, D15, D16, D17, D18, D19, D2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
