File: top_plate/therick64BA_top_plate.kicad_pcb (KiCad board)
At the start: 2 copper layers, 313.5 x 75.4 mm, 74 parts, among them U1 HOLE, U10 HOLE, U11 HOLE, U12 HOLE, U13 HOLE, U14 HOLE, U15 HOLE, U16 HOLE, U17 HOLE, U18 HOLE, U19 HOLE, U2 HOLE, U20 HOLE, U21 HOLE, U22 HOLE, U23 HOLE, U24 HOLE, U25 HOLE, U26 HOLE, U27 HOLE, U28 HOLE, U29 HOLE, U3 HOLE, U30 HOLE, U31 HOLE, U32 HOLE, U33 HOLE, U34 HOLE, U35 HOLE, U36 HOLE, U37 HOLE, U38 HOLE, U39 HOLE, U4 HOLE, U40 HOLE, U41 HOLE, U42 HOLE, U43 HOLE, U44 HOLE, U45 HOLE, U46 HOLE, U47 HOLE, U48 HOLE, U49 HOLE, U5 HOLE, U50 HOLE, U51 HOLE, U52 HOLE, U53 HOLE, U54 HOLE, U55 HOLE, U56 HOLE, U57 HOLE, U58 HOLE, U59 HOLE, U6 HOLE, U60 HOLE, U61 HOLE, U62 HOLE, U63 HOLE, U64 HOLE, U7 HOLE, U8 HOLE, U9 HOLE

Commit message: Update to 19mm
Parts:
- added U65: HOLE, acheron_Hardware:MouseBite_IPC7351, F.Cu at (273.6, 91.6)
- added U66: HOLE, acheron_Hardware:MouseBite_IPC7351, F.Cu at (273.2, 72.6)
- added U67: HOLE, acheron_Hardware:MouseBite_IPC7351, F.Cu at (273.6, 53.6)
- moved U48 0.82 mm to (264.5, 101.1)
- moved U36 0.79 mm to (264.5, 82.1)
- moved U47 0.78 mm to (245.5, 101.1)
- moved H6 0.77 mm to (254.9, 74.6)
- moved U24 0.76 mm to (264.5, 63.1)
- moved U11 0.75 mm to (245.5, 44.1)
- moved U35 0.75 mm to (245.5, 82.1)
- moved U46 0.74 mm to (226.5, 101.1)
- moved U12 0.73 mm to (264.5, 44.1)
- moved U23 0.72 mm to (245.5, 63.1)
- moved H5 0.71 mm to (216.9, 93.6)
- moved U34 0.71 mm to (226.5, 82.1)
- moved U45 0.71 mm to (207.5, 101.1)
- moved U64 0.71 mm to (350.4, 101.1)
- moved U22 0.68 mm to (226.5, 63.1)
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Other:
- board size 313.5 x 75.4 mm -> 313.1 x 75.2 mm
- board text added: "therick64BA_19mm"

Commit message: Changed pins to make routing cleaner
Other:
- board text added: "therick64BA Rev 1.0"
- board text removed: "therick64BA_19mm"
