File: top_plate/therick48.16_top_plate.kicad_pcb (KiCad board)
At the start: 2 copper layers, 309.7 x 75.2 mm, 85 parts, among them U1 HOLE, U10 HOLE, U11 HOLE, U12 HOLE, U13 HOLE, U14 HOLE, U15 HOLE, U16 HOLE, U17 HOLE, U18 HOLE, U19 HOLE, U2 HOLE, U20 HOLE, U21 HOLE, U22 HOLE, U23 HOLE, U24 HOLE, U25 HOLE, U26 HOLE, U27 HOLE, U28 HOLE, U29 HOLE, U3 HOLE, U30 HOLE, U31 HOLE, U32 HOLE, U33 HOLE, U34 HOLE, U35 HOLE, U36 HOLE, U37 HOLE, U38 HOLE, U39 HOLE, U4 HOLE, U40 HOLE, U41 HOLE, U42 HOLE, U43 HOLE, U44 HOLE, U45 HOLE, U46 HOLE, U47 HOLE, U48 HOLE, U49 HOLE, U5 HOLE, U50 HOLE, U51 HOLE, U52 HOLE, U53 HOLE, U54 HOLE, U55 HOLE, U56 HOLE, U57 HOLE, U58 HOLE, U59 HOLE, U6 HOLE, U60 HOLE, U61 HOLE, U62 HOLE, U63 HOLE, U64 HOLE, U65 HOLE, U66 HOLE, U67 HOLE, U7 HOLE, U8 HOLE, U9 HOLE

Commit message: 48+16 to 48.16
Other:
- board text added: "therick48.16 Rev 1.0"
- board text removed: "therick48+16 Rev 1.0"
Changed lines of the file:
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@@
   (gr_arc (start 274.74 87.4) (end 273.6 87.4) (angle -180) (layer Edge.Cuts) (width 0.05))
   (gr_arc (start 274.74 95.76) (end 275.88 95.76) (angle -180) (layer Edge.Cuts) (width 0.05))
-  (gr_text "therick48+16 Rev 1.0" (at 159.98 91.58) (layer B.SilkS)
+  (gr_text "therick48.16 Rev 1.0" (at 159.98 91.58) (layer B.SilkS)
     (effects (font (size 1.5 1.5) (thickness 0.2)) (justify mirror))
   )
