File: 03 bottom_plate/therick48.16_bottom_plate.kicad_pcb (KiCad board)
At the start: 2 copper layers, 310.5 x 76 mm, 88 parts, among them U1 HOLE, U10 HOLE, U11 HOLE, U12 HOLE, U13 HOLE, U14 HOLE, U15 HOLE, U16 HOLE, U17 HOLE, U18 HOLE, U19 HOLE, U2 HOLE, U20 HOLE, U21 HOLE, U22 HOLE, U23 HOLE, U24 HOLE, U25 HOLE, U26 HOLE, U27 HOLE, U28 HOLE, U29 HOLE, U3 HOLE, U30 HOLE, U31 HOLE, U32 HOLE, U33 HOLE, U34 HOLE, U35 HOLE, U36 HOLE, U37 HOLE, U38 HOLE, U39 HOLE, U4 HOLE, U40 HOLE, U41 HOLE, U42 HOLE, U43 HOLE, U44 HOLE, U45 HOLE, U46 HOLE, U47 HOLE, U48 HOLE, U49 HOLE, U5 HOLE, U50 HOLE, U51 HOLE, U52 HOLE, U53 HOLE, U54 HOLE, U55 HOLE, U56 HOLE, U57 HOLE, U58 HOLE, U59 HOLE, U6 HOLE, U60 HOLE, U61 HOLE, U62 HOLE, U63 HOLE, U64 HOLE, U65 HOLE, U66 HOLE, U67 HOLE, U68 HOLE, U69 HOLE, U7 HOLE, U70 HOLE, U8 HOLE, U9 HOLE

Commit message: Add reset hole to bottom plate
Parts:
- added H19: MountingHole, random-keyboard-parts:Generic-Mounthole, F.Cu at (103.4, 46.0)
Changed lines of the file:
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@@
     (tracks 0)
     (zones 0)
-    (modules 88)
+    (modules 89)
     (nets 1)
   )
@@
   )
   (module random-keyboard-parts:Generic-Mounthole (layer F.Cu)
+    (at 103.359728 45.979879)
+    (attr virtual)
+    (fp_text reference H19 (at 0 2) (layer Dwgs.User)
+      (effects (font (size 1 1) (thickness 0.15)))
+    )
+    (fp_text value MountingHole (at 0 -2) (layer Dwgs.User)
+      (effects (font (size 1 1) (thickness 0.15)))
+    )
+    (pad 1 thru_hole circle (at 0 0) (size 3.5 3.5) (drill 2.2) (layers *.Cu *.Mask))
+  )
+  (module random-keyboard-parts:Generic-Mounthole (layer F.Cu)
