File: 01 PCB/therick48.16.sch (KiCad schematic (older format))
At the start: 173 parts, among them J1 TYPE-C-31-M12_13, J2 AVR-ISP-6_mod, K1 KEYSW, K10 KEYSW, K11 KEYSW, K12 KEYSW, K13 KEYSW, K14 KEYSW, K15 KEYSW, K16 KEYSW, K17 KEYSW, K18 KEYSW, K19 KEYSW, K2 KEYSW, K20 KEYSW, K21 KEYSW, K22 KEYSW, K23 KEYSW, K24 KEYSW, K25 KEYSW, K26 KEYSW, K27 KEYSW, K28 KEYSW, K29 KEYSW, K3 KEYSW, K30 KEYSW, K31 KEYSW, K32 KEYSW, K33 KEYSW, K34 KEYSW, K35 KEYSW, K36 KEYSW, K37 KEYSW, K38 KEYSW, K39 KEYSW, K4 KEYSW, K40 KEYSW, K41 KEYSW, K42 KEYSW, K43 KEYSW, K44 KEYSW, K45 KEYSW, K46 KEYSW, K47 KEYSW, K48 KEYSW, K49 KEYSW, K5 KEYSW, K50 KEYSW, K51 KEYSW, K52 KEYSW, K53 KEYSW, K54 KEYSW, K55 KEYSW, K56 KEYSW, K57 KEYSW, K58 KEYSW, K59 KEYSW, K6 KEYSW, K60 KEYSW, K61 KEYSW, K62 KEYSW, K63 KEYSW, K64 KEYSW, K7 KEYSW, K8 KEYSW, K9 KEYSW, SW1 SW_PUSH, U1 ATMEGA32U4, U2 HOLE, U3 USBLC6-2SC6, U4 HOLE, U5 HOLE, U6 HOLE, U7 HOLE, U8 HOLE, Y1 16MHz

Commit message: Update 04 Schematic.png
Other:
- note added: ".16 Holes"
- note removed: "+16 Holes"
Changed lines of the file:
@@
 EESchema Schematic File Version 4
-LIBS:therick64BA-cache
+LIBS:therick48.16-cache
 EELAYER 29 0
 EELAYER END
@@
 	12350 4500 11050 4500
 Text Notes 11300 6550 0    50   ~ 0
-+16 Holes
+.16 Holes
 Wire Notes Line
 	11050 5600 11900 5600

Commit message: Add Power LED
Parts:
- added LED1: LED, LED_SMD:LED_0805_2012Metric_Pad1.15x1.40mm_HandSolder, symbol keyboard_parts:LED
- added R4: 1K, Resistor_SMD:R_0805_2012Metric_Pad1.15x1.40mm_HandSolder, symbol Device:R_Small
- added U9: HOLE, Symbol:OSHW-Logo2_9.8x8mm_SilkScreen, symbol lets_split-cache:HOLE
Connections:
- net GND: now also LED1.1 (K)
- net VCC: now also R4.2
- new net: LED1.2 (A), R4.1
Other:
- note added: "Open Hardware"
- note added: "Power LED"
- note added: "THERICK"
- moved on the sheet: U2, U8
Changed lines of the file:
@@
 L lets_split-cache:HOLE U2
 U 1 1 5DE56E92
-P 9400 4250
-F 0 "U2" H 9578 4303 60  0000 L CNN
-F 1 "HOLE" H 9578 4197 60  0000 L CNN
-F 2 "Artwork:rick_large" H 9400 4250 60  0001 C CNN
-F 3 "" H 9400 4250 60  0001 C CNN
-	1    9400 4250
+P 9300 7000
+F 0 "U2" H 9478 7053 60  0000 L CNN
+F 1 "HOLE" H 9478 6947 60  0000 L CNN
+F 2 "Artwork:rick_large" H 9300 7000 60  0001 C CNN
+F 3 "" H 9300 7000 60  0001 C CNN
+	1    9300 7000
 	1    0    0    -1
 $EndComp
@@
 Text Notes 9600 5400 0    50   ~ 0
 Planck Holes
-Text Notes 9250 4500 0    50   ~ 0
+Text Notes 9150 7250 0    50   ~ 0
 Graphic
 Wire Notes Line
-	9200 4550 9200 4050
-Wire Notes Line
-	9200 4050 9850 4050
-Wire Notes Line
-	9850 4050 9850 4550
-Wire Notes Line
-	9850 4550 9200 4550
+	9100 7300 9100 6800
+Wire Notes Line
+	9100 6800 9750 6800
+Wire Notes Line
+	9750 6800 9750 7300
+Wire Notes Line
+	9750 7300 9100 7300
 Text GLabel 2050 5500 2    50   BiDi ~ 0
 D+BUS
@@
 	1    0    0    -1
 $EndComp
-Text Notes 11400 5400 0    50   ~ 0
-Mouse bites
 Wire Notes Line
 	11050 4500 11050 5450
 Wire Notes Line
 	11050 5450 12350 5450
-Wire Notes Line
-	12350 5450 12350 4500
 Wire Notes Line
 	12350 4500 11050 4500
@@
 L lets_split-cache:HOLE U8
 U 1 1 5F0F74C2
-P 10150 4250
-F 0 "U8" H 10328 4303 60  0000 L CNN
-F 1 "HOLE" H 10328 4197 60  0000 L CNN
-F 2 "Artwork:THERICK" H 10150 4250 60  0001 C CNN
-F 3 "" H 10150 4250 60  0001 C CNN
-	1    10150 4250
-	1    0    0    -1
-$EndComp
-Text Notes 10000 4500 0    50   ~ 0
-Graphic
-Wire Notes Line
-	9950 4550 9950 4050
-Wire Notes Line
-	9950 4050 10600 4050
-Wire Notes Line
-	10600 4050 10600 4550
-Wire Notes Line
-	10600 4550 9950 4550
+P 10050 7000
+F 0 "U8" H 10228 7053 60  0000 L CNN
+F 1 "HOLE" H 10228 6947 60  0000 L CNN
+F 2 "Artwork:THERICK" H 10050 7000 60  0001 C CNN
+F 3 "" H 10050 7000 60  0001 C CNN
+	1    10050 7000
+	1    0    0    -1
+$EndComp
+Text Notes 9900 7250 0    50   ~ 0
+THERICK
+Wire Notes Line
+	9850 7300 9850 6800
+Wire Notes Line
+	9850 6800 10500 6800
+Wire Notes Line
+	10500 6800 10500 7300
+Wire Notes Line
+	10500 7300 9850 7300
+$Comp
+L power:VCC #PWR0126
+U 1 1 5FB518F2
+P 1250 8000
+F 0 "#PWR0126" H 1250 7850 50  0001 C CNN
+F 1 "VCC" V 1268 8127 50  0000 L CNN
+F 2 "" H 1250 8000 50  0001 C CNN
+F 3 "" H 1250 8000 50  0001 C CNN
+	1    1250 8000
+	0    -1   -1   0
+$EndComp
+$Comp
+L keyboard_parts:LED LED1
+U 1 1 5FB52A4E
+P 1750 8000
+F 0 "LED1" H 1750 7850 30  0000 C CNN
+F 1 "LED" H 1750 7900 30  0000 C CNN
+F 2 "LED_SMD:LED_0805_2012Metric_Pad1.15x1.40mm_HandSolder" H 1750 8000 60  0001 C CNN
+F 3 "" H 1750 8000 60  0000 C CNN
+	1    1750 8000
+	-1   0    0    1
+$EndComp
+$Comp
+L Device:R_Small R4
+U 1 1 5FB53F04
+P 1400 8000
+F 0 "R4" V 1300 8000 30  0000 C CNN
+F 1 "1K" V 1400 8000 30  0000 C CNN
+F 2 "Resistor_SMD:R_0805_2012Metric_Pad1.15x1.40mm_HandSolder" H 1400 8000 50  0001 C CNN
+F 3 "~" H 1400 8000 50  0001 C CNN
+	1    1400 8000
+	0    1    1    0
+$EndComp
+$Comp
+L power:GND #PWR0127
+U 1 1 5FB5552C
+P 2000 8000
+F 0 "#PWR0127" H 2000 7750 50  0001 C CNN
+F 1 "GND" V 2005 7872 50  0000 R CNN
+F 2 "" H 2000 8000 50  0001 C CNN
+F 3 "" H 2000 8000 50  0001 C CNN
+	1    2000 8000
+	0    -1   -1   0
+$EndComp
+Wire Wire Line
+	2000 8000 1950 8000
+Wire Wire Line
+	1550 8000 1500 8000
+Wire Wire Line
+	1300 8000 1250 8000
+Text Notes 1450 8150 0    50   ~ 0
+Power LED
+Wire Notes Line
+	2300 8200 950  8200
+Wire Notes Line
+	950  8200 950  7800
+Wire Notes Line
+	950  7800 2300 7800
+Wire Notes Line
+	2300 7800 2300 8200
+$Comp
+L lets_split-cache:HOLE U9
+U 1 1 5FC72ADE
+P 10800 7000
+F 0 "U9" H 10978 7053 60  0000 L CNN
+F 1 "HOLE" H 10978 6947 60  0000 L CNN
+F 2 "Symbol:OSHW-Logo2_9.8x8mm_SilkScreen" H 10800 7000 60  0001 C CNN
+F 3 "" H 10800 7000 60  0001 C CNN
+	1    10800 7000
+	1    0    0    -1
+$EndComp
+Text Notes 10650 7250 0    50   ~ 0
+Open Hardware
+Wire Notes Line
+	10600 7300 10600 6800
+Wire Notes Line
+	10600 6800 11250 6800
+Wire Notes Line
+	11250 6800 11250 7300
+Wire Notes Line
+	11250 7300 10600 7300
+Text Notes 11400 5400 0    50   ~ 0
+Mouse bites
+Wire Notes Line
+	12350 5450 12350 4500
 $EndSCHEMATC
